File: diagrams/voltage_dividers.kicad_sch (KiCad schematic)
At the start: 8 parts, among them J1 3.3v Output, J2 5v Input, J3 80v Input, J4 5v Output

Commit message: docs & diagrams
Parts:
- R3: value 150k -> 1M
- R4: value 10k -> 68k
Changed lines of the file:
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@@
 			)
 		)
-		(property "Value" "150k"
+		(property "Value" "1M"
 			(at 93.98 20.3199 0)
 			(effects
@@
 			)
 		)
-		(property "Value" "10k"
+		(property "Value" "68k"
 			(at 93.98 30.4799 0)
 			(effects
