File: diagrams/modules.kicad_sch (KiCad schematic)
At the start: 20 parts, among them U1 MCU, U10 MCU 3.3v, U11 Hall 5v, U12 NRF52840, U13 Buck Converter, U2 ADS1115, U3 Throttle, U4 Controller, U5 Hall 5v, U6 MCU 3.3v, U7 MCU 3.3v, U8 Controller, U9 Brake 5v

Commit message: svg diagrams
Connections:
- net at U8. (SIG), U9. (SIG): now also R4.2, U7. (SIG); no longer R3.2
- net at U3. (SIG): now also U4. (SIG); no longer U2. (VDD)
- net at U4. (SIG): now also U?. (VOUT); no longer U3. (SIG)
- new net: R3.2, U8. (SIG), U9. (SIG)
- new net: U1. (SDA), U2. (VDD), U3. (SIG), U4. (SIG), U?. (VOUT)
- new net: U1. (SDA), U2. (VDD), U?. (VOUT) (x3)
- new net: U2. (VDD), U3. (SIG)
- now unconnected: U2. (VDD), U2. (VDD), U2. (VDD), U2. (VDD)
Changed lines of the file:
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@@
 	(generator "eeschema")
 	(generator_version "8.0")
-	(paper "A5")
+	(paper "A4")
 	(title_block
 		(title "modules")
